File: Eagle/projects/xPi.brd (EAGLE design)
At the start: 64.4 x 91.4 mm, 37 parts, among them T1 BC337, T2 BC337, T3 BC337

Commit message: xPi v1.4
Parts:
- removed SG1: F/CM12P, buzzer:F/CM12P
- added D4, D5: 1N4004, diode:DO41-10
- added SG5: F/CM12P, buzzer:F/CM12P
- R6, R7, R8, R9: value 480 -> 470
- renumbered +12V- to +15V-
Connections:
- new net N$8: +15V-.2, D4.A
- new net N$9: D5.A, U$5.VO
- net +12V: now also D4.C; no longer +15V-.2
- net +5V: now also D5.C, SG5.+; no longer SG1.+, U$5.VO
- net N$4: now also SG5.-; no longer SG1.-
Routing:
- net N$8: track 0.00 -> 13.7 mm
- net N$9: track 0.00 -> 6.13 mm
- net +12V: track 99.1 -> 93.0 mm
- net N$4: track 11.2 -> 9.94 mm
Other:
- board size 64.4 x 91.4 mm -> 64.4 x 92.7 mm
- board text added: "Regulate Voltage to 5.6V"
- board text added: "xPi v1.4 2018"
- board text removed: "xPi v1.3 2018"
