File: Eagle/projects/xPi.sch (EAGLE design)
At the start: 37 parts, among them T1 BC337, T2 BC337, T3 BC337

Commit message: xPi v1.4
Parts:
- added D4, D5: 1N4004, diode:1N4004
- R6, R7, R8, R9: value 480 -> 470
- renumbered +12V- to +15V-, SG1 to SG5
Connections:
- new net N$8: +15V--2.KL, D4.A
- new net N$9: D5.A, U$5.VO
- net +12V: now also D4.C; no longer +15V--2.KL
- net +5V: now also D5.C; no longer U$5.VO
Changed lines of the file:
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@@
 <part name="R1" library="resistor" library_urn="urn:adsk.eagle:library:348" deviceset="R-EU_" device="0204/7" package3d_urn="urn:adsk.eagle:package:25945/1" value="1K2"/>
 <part name="GND6" library="supply1" library_urn="urn:adsk.eagle:library:371" deviceset="GND" device=""/>
-<part name="+12V-" library="con-ptr500" library_urn="urn:adsk.eagle:library:181" deviceset="AK300/2" device="" package3d_urn="urn:adsk.eagle:package:9881/1" value="Alim+15v"/>
+<part name="+15V-" library="con-ptr500" library_urn="urn:adsk.eagle:library:181" deviceset="AK300/2" device="" package3d_urn="urn:adsk.eagle:package:9881/1" value="Alim+15v"/>
 <part name="D3" library="diode" library_urn="urn:adsk.eagle:library:210" deviceset="1N4004" device="" package3d_urn="urn:adsk.eagle:package:43336/1"/>
 <part name="P+6" library="supply1" library_urn="urn:adsk.eagle:library:371" deviceset="+12V" device=""/>
@@
 <part name="P+8" library="supply1" library_urn="urn:adsk.eagle:library:371" deviceset="+12V" device=""/>
 <part name="GND7" library="supply1" library_urn="urn:adsk.eagle:library:371" deviceset="GND" device=""/>
-<part name="R6" library="rcl" library_urn="urn:adsk.eagle:library:334" deviceset="R-EU_" device="0204/7" package3d_urn="urn:adsk.eagle:package:23498/1" value="480"/>
-<part name="R7" library="rcl" library_urn="urn:adsk.eagle:library:334" deviceset="R-EU_" device="0204/7" package3d_urn="urn:adsk.eagle:package:23498/1" value="480"/>
-<part name="R8" library="rcl" library_urn="urn:adsk.eagle:library:334" deviceset="R-EU_" device="0204/7" package3d_urn="urn:adsk.eagle:package:23498/1" value="480"/>
-<part name="R9" library="rcl" library_urn="urn:adsk.eagle:library:334" deviceset="R-EU_" device="0204/7" package3d_urn="urn:adsk.eagle:package:23498/1" value="480"/>
+<part name="R6" library="rcl" library_urn="urn:adsk.eagle:library:334" deviceset="R-EU_" device="0204/7" package3d_urn="urn:adsk.eagle:package:23498/1" value="470"/>
+<part name="R7" library="rcl" library_urn="urn:adsk.eagle:library:334" deviceset="R-EU_" device="0204/7" package3d_urn="urn:adsk.eagle:package:23498/1" value="470"/>
+<part name="R8" library="rcl" library_urn="urn:adsk.eagle:library:334" deviceset="R-EU_" device="0204/7" package3d_urn="urn:adsk.eagle:package:23498/1" value="470"/>
+<part name="R9" library="rcl" library_urn="urn:adsk.eagle:library:334" deviceset="R-EU_" device="0204/7" package3d_urn="urn:adsk.eagle:package:23498/1" value="470"/>
 <part name="R11" library="resistor" library_urn="urn:adsk.eagle:library:348" deviceset="R-EU_" device="0204/7" package3d_urn="urn:adsk.eagle:package:25945/1" value="680"/>
 <part name="U$5" library="DSWY2596" deviceset="DSWY2596" device=""/>
@@
 <part name="P" library="pinhead" library_urn="urn:adsk.eagle:library:325" deviceset="PINHD-1X6" device="" package3d_urn="urn:adsk.eagle:package:22472/2"/>
 <part name="GND18" library="supply1" library_urn="urn:adsk.eagle:library:371" deviceset="GND" device=""/>
-<part name="SG1" library="buzzer" library_urn="urn:adsk.eagle:library:113" deviceset="F/CM12P" device="" package3d_urn="urn:adsk.eagle:package:5265/1"/>
+<part name="D4" library="diode" library_urn="urn:adsk.eagle:library:210" deviceset="1N4004" device="" package3d_urn="urn:adsk.eagle:package:43336/1"/>
+<part name="D5" library="diode" library_urn="urn:adsk.eagle:library:210" deviceset="1N4004" device="" package3d_urn="urn:adsk.eagle:package:43336/1"/>
+<part name="SG5" library="buzzer" library_urn="urn:adsk.eagle:library:113" deviceset="F/CM12P" device="" package3d_urn="urn:adsk.eagle:package:5265/1"/>
 </parts>
 <sheets>
@@
 <instance part="+BATT-" gate="-1" x="83.82" y="-66.04" rot="R180"/>
 <instance part="+BATT-" gate="-2" x="83.82" y="-60.96" rot="R180"/>
-<instance part="P+4" gate="1" x="-12.7" y="-40.64"/>
+<instance part="P+4" gate="1" x="-12.7" y="-35.56"/>
 <instance part="R2" gate="G$1" x="-38.1" y="17.78" rot="R180"/>
 <instance part="GND5" gate="1" x="-12.7" y="-27.94" rot="MR0"/>
 <instance part="R1" gate="G$1" x="-27.94" y="-15.24" rot="MR0"/>
 <instance part="GND6" gate="1" x="63.5" y="-71.12"/>
-<instance part="+12V-" gate="-1" x="58.42" y="-66.04"/>
-<instance part="+12V-" gate="-2" x="58.42" y="-33.02"/>
+<instance part="+15V-" gate="-1" x="58.42" y="-66.04"/>
+<instance part="+15V-" gate="-2" x="58.42" y="-33.02"/>
 <instance part="D3" gate="1" x="86.36" y="-48.26" rot="R90"/>
 <instance part="P+6" gate="1" x="96.52" y="-30.48"/>
@@
 <instance part="P" gate="A" x="-63.5" y="-88.9" rot="MR0"/>
 <instance part="GND18" gate="1" x="-53.34" y="-96.52"/>
-<instance part="SG1" gate="G$1" x="-7.62" y="-5.08" rot="R270"/>
+<instance part="D4" gate="1" x="68.58" y="-33.02"/>
+<instance part="D5" gate="1" x="-12.7" y="-45.72" rot="R90"/>
+<instance part="SG5" gate="G$1" x="-7.62" y="-5.08" rot="R270"/>
 </instances>
 <busses>
@@
 <nets>
 <net name="+5V" class="0">
-<segment>
-<pinref part="U$5" gate="G$1" pin="VO"/>
-<pinref part="P+4" gate="1" pin="+5V"/>
-<wire x1="-12.7" y1="-43.18" x2="-12.7" y2="-50.8" width="0.1524" layer="91"/>
-</segment>
 <segment>
 <pinref part="U$6" gate="G$1" pin="5V@2"/>
@@
 <pinref part="P+2" gate="1" pin="+5V"/>
 <wire x1="-10.16" y1="-2.54" x2="-12.7" y2="-2.54" width="0.1524" layer="91"/>
-<pinref part="SG1" gate="G$1" pin="1"/>
+<pinref part="SG5" gate="G$1" pin="1"/>
+</segment>
+<segment>
+<pinref part="P+4" gate="1" pin="+5V"/>
+<pinref part="D5" gate="1" pin="C"/>
+<wire x1="-12.7" y1="-38.1" x2="-12.7" y2="-43.18" width="0.1524" layer="91"/>
 </segment>
 </net>
@@
 <pinref part="+BATT-" gate="-1" pin="KL"/>
 <wire x1="78.74" y1="-66.04" x2="63.5" y2="-66.04" width="0.1524" layer="91"/>
-<pinref part="+12V-" gate="-1" pin="KL"/>
+<pinref part="+15V-" gate="-1" pin="KL"/>
 <junction x="63.5" y="-66.04"/>
 <wire x1="63.5" y1="-66.04" x2="63.5" y2="-68.58" width="0.1524" layer="91"/>
@@
 <wire x1="86.36" y1="-33.02" x2="96.52" y2="-33.02" width="0.1524" layer="91"/>
 <pinref part="P+6" gate="1" pin="+12V"/>
+<pinref part="D4" gate="1" pin="C"/>
+<pinref part="F1" gate="G$1" pin="2"/>
+<wire x1="71.12" y1="-33.02" x2="78.74" y2="-33.02" width="0.1524" layer="91"/>
+<wire x1="78.74" y1="-33.02" x2="86.36" y2="-33.02" width="0.1524" layer="91"/>
+<junction x="78.74" y="-33.02"/>
 <junction x="86.36" y="-33.02"/>
-<pinref part="F1" gate="G$1" pin="2"/>
-<wire x1="63.5" y1="-33.02" x2="86.36" y2="-33.02" width="0.1524" layer="91"/>
-<pinref part="+12V-" gate="-2" pin="KL"/>
-<junction x="63.5" y="-33.02"/>
-<wire x1="63.5" y1="-33.02" x2="78.74" y2="-33.02" width="0.1524" layer="91"/>
 </segment>
 <segment>
@@
 <pinref part="T3" gate="G$1" pin="C"/>
 <wire x1="-10.16" y1="-10.16" x2="-12.7" y2="-10.16" width="0.1524" layer="91"/>
-<pinref part="SG1" gate="G$1" pin="2"/>
+<pinref part="SG5" gate="G$1" pin="2"/>
 </segment>
 </net>
@@
 </segment>
 </net>
+<net name="N$8" class="0">
+<segment>
+<pinref part="+15V-" gate="-2" pin="KL"/>
+<pinref part="D4" gate="1" pin="A"/>
+<wire x1="66.04" y1="-33.02" x2="63.5" y2="-33.02" width="0.1524" layer="91"/>
+</segment>
+</net>
+<net name="N$9" class="0">
+<segment>
+<pinref part="U$5" gate="G$1" pin="VO"/>
+<pinref part="D5" gate="1" pin="A"/>
+<wire x1="-12.7" y1="-48.26" x2="-12.7" y2="-50.8" width="0.1524" layer="91"/>
+</segment>
+</net>
